File: UniSeb32.kicad_sch (KiCad schematic)
At the start: 57 parts, among them J1 IO, J2 ARJM11C7-114-BA-EW2, J3 Conn_02x05_Odd_Even, J6 SDS011, J7 Conn_01x02_Female, J8 Conn_01x02_Female, U1 mini_esp32, U2 LAN8720A, U3 AMS1117-3.3, U4 AMS5919, U5 module_bme280, U6 RT9400, U7 MCP23008-xSS, U8 HLK-PM01, X1 233-508, X2 233-503, X3 233-504, Y1 Crystal_GND23

Commit message: Added attributes for jlcpcb assembly
Parts:
- C10, C13, C4: JLC (none) -> 0603; LCSC (none) -> C14663; jlcpcb C14663 -> (none)
- C11: JLC (none) -> 0603; LCSC (none) -> C57112; jlcpcb C57112 -> (none)
- C12: JLC (none) -> 0603; LCSC (none) -> C23630; jlcpcb C23630 -> (none)
- C14, C15: JLC (none) -> 0603; LCSC (none) -> C1658; jlcpcb C1658 -> (none)
- C3: JLC (none) -> 1206; LCSC (none) -> C5672; jlcpcb C5672 -> (none)
- C5, C6, C7, C8: JLC (none) -> 0603; LCSC (none) -> C1634; jlcpcb C1634 -> (none)
- C9: JLC (none) -> 0603; LCSC (none) -> C96446; jlcpcb C96446 -> (none)
- L1: JLC (none) -> 0805; LCSC (none) -> C1017
- R10, R11, R13, R9: JLC (none) -> 0603; LCSC (none) -> C23185
- R12, R8: JLC (none) -> 0603; LCSC (none) -> C4190; jlcpcb C22938 -> (none)
- R14: JLC (none) -> 0603; LCSC (none) -> C22790; jlcpcb C269454 -> (none)
- R15, R16, R17, R18, R19, R20, R4: JLC (none) -> 0603; LCSC (none) -> C25804; jlcpcb C25197 -> (none)
- R2: JLC (none) -> 0603; LCSC (none) -> C21189
- R5: JLC (none) -> 0603; LCSC (none) -> C23162; jlcpcb C23162 -> (none)
- U2: JLC (none) -> QFN24; LCSC (none) -> C45223
- U3: JLC (none) -> SOT223-3; LCSC (none) -> C6186
- Y1: JLC (none) -> 3225; LCSC (none) -> C9006; jlcpcb C9006 -> (none)
