File: UniSeb32.kicad_sch (KiCad schematic)
At the start: 56 parts, among them J1 IO, J101 Micro_SD_Card_Det, J2 ARJM11C7-114-BA-EW2, J3 Conn_02x05_Odd_Even, J6 SDS011, J7 Conn_01x02_Female, J8 Conn_01x02_Female, U1 mini_esp32, U2 LAN8720A, U3 AMS1117-3.3, U4 AMS5915, U5 module_bme280, U6 RT9400, U7 MCP23008-xSS, U8 HLK-PM01, X1 233-508, X2 233-503, X3 233-504

Commit message: .
Parts:
- added C15: 1n, Capacitor_SMD:C_0603_1608Metric, symbol Device:C_Small
Connections:
- net GND: now also C15.2
- net RX_P: now reaches C7.2, J2.5 (RD+), R11.2, U2.23 (RXP)
- net TX_N: now reaches C6.1, J2.8 (TD-), R10.2, U2.20 (TXN)
- net TX_P: now reaches C5.1, J2.10 (TD+), R9.2, U2.21 (TXP)
- net RX_N: now reaches C8.1, J2.3 (RD-), R13.2, U2.22 (RXN)
- net at C14.1: now also J2.SH2 (SHIELD); no longer J2.SH (SHIELD)
- new net: C15.1, J2.SH1 (SHIELD)
Changed lines of the file:
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@@
   (junction (at 162.56 180.34) (diameter 0) (color 0 0 0 0)
   )
+  (junction (at 91.44 325.12) (diameter 0) (color 0 0 0 0)
+  )
   (junction (at 181.61 325.12) (diameter 0) (color 0 0 0 0)
   )
@@
     (stroke (width 0) (type default) (color 0 0 0 0))
   )
+  (wire (pts (xy 91.44 313.69) (xy 91.44 317.5))
+    (stroke (width 0) (type default) (color 0 0 0 0))
+  )
   (wire (pts (xy 138.43 270.51) (xy 138.43 281.94))
     (stroke (width 0) (type default) (color 0 0 0 0))
@@
     (stroke (width 0) (type default) (color 0 0 0 0))
   )
+  (wire (pts (xy 83.185 311.15) (xy 83.185 317.5))
+    (stroke (width 0) (type default) (color 0 0 0 0))
+  )
   (wire (pts (xy 187.325 43.18) (xy 193.04 43.18))
     (stroke (width 0) (type default) (color 0 0 0 0))
@@
     (stroke (width 0) (type default) (color 0 0 0 0))
   )
+  (wire (pts (xy 83.185 322.58) (xy 83.185 325.12))
+    (stroke (width 0) (type default) (color 0 0 0 0))
+  )
   (wire (pts (xy 97.79 130.81) (xy 97.79 128.27))
     (stroke (width 0) (type default) (color 0 0 0 0))
@@
     (stroke (width 0) (type default) (color 0 0 0 0))
   )
+  (wire (pts (xy 91.44 311.15) (xy 83.185 311.15))
+    (stroke (width 0) (type default) (color 0 0 0 0))
+  )
   (wire (pts (xy 162.56 187.96) (xy 152.4 187.96))
     (stroke (width 0) (type default) (color 0 0 0 0))
@@
     (stroke (width 0) (type default) (color 0 0 0 0))
   )
-  (wire (pts (xy 91.44 311.15) (xy 91.44 317.5))
-    (stroke (width 0) (type default) (color 0 0 0 0))
-  )
   (wire (pts (xy 78.74 53.34) (xy 80.01 53.34))
     (stroke (width 0) (type default) (color 0 0 0 0))
@@
     (stroke (width 0) (type default) (color 0 0 0 0))
   )
+  (wire (pts (xy 83.185 325.12) (xy 91.44 325.12))
+    (stroke (width 0) (type default) (color 0 0 0 0))
+  )
   (wire (pts (xy 157.48 182.88) (xy 149.86 182.88))
     (stroke (width 0) (type default) (color 0 0 0 0))
@@
     (effects (font (size 0.7112 0.7112)) (justify right bottom))
   )
+  (label "TX_N" (at 153.67 284.48 0)
+    (effects (font (size 1.27 1.27)) (justify left bottom))
+  )
   (label "EMAC_TXD0" (at 198.12 289.56 0)
     (effects (font (size 1.27 1.27)) (justify left bottom))
@@
     (effects (font (size 1.27 1.27)) (justify right bottom))
   )
+  (label "TX_P" (at 153.67 287.02 0)
+    (effects (font (size 1.27 1.27)) (justify left bottom))
+  )
   (label "SDS_TX" (at 124.46 157.48 270)
     (effects (font (size 0.7112 0.7112)) (justify right bottom))
@@
     (effects (font (size 1.27 1.27)) (justify left bottom))
   )
+  (label "RX_N" (at 153.67 279.4 0)
+    (effects (font (size 1.27 1.27)) (justify left bottom))
+  )
   (label "EMAC_RXD1" (at 55.245 189.23 180)
     (effects (font (size 1.27 1.27)) (justify right bottom))
@@
     (effects (font (size 1.27 1.27)) (justify left bottom))
   )
+  (label "RX_P" (at 153.67 281.94 0)
+    (effects (font (size 1.27 1.27)) (justify left bottom))
+  )
   (label "SCMD" (at 93.98 182.245 180)
     (effects (font (size 1.27 1.27)) (justify right bottom))
@@
     (pin "8")
     (pin "9")
-    (pin "SH")
+    (pin "SH1")
+    (pin "SH2")
   )
   (symbol (lib_id "power:GND") (at 81.28 60.96 0) (unit 1)
@@
     (pin "1")
   )
+  (symbol (lib_id "Device:C_Small") (at 83.185 320.04 0) (unit 1)
+    (in_bom yes) (on_board yes)
+    (property "Reference" "C15" (id 0) (at 79.375 318.77 0)
+      (effects (font (size 1.27 1.27)) (justify left))
+    )
+    (property "Value" "1n" (id 1) (at 76.835 321.31 0)
+      (effects (font (size 1.27 1.27)) (justify left))
+    )
+    (property "Footprint" "Capacitor_SMD:C_0603_1608Metric" (id 2) (at 83.185 320.04 0)
+      (effects (font (size 1.27 1.27)) hide)
+    )
+    (property "Datasheet" "~" (id 3) (at 83.185 320.04 0)
+      (effects (font (size 1.27 1.27)) hide)
+    )
+    (property "LCSC" "C9196" (id 4) (at 83.185 320.04 0)
+      (effects (font (size 1.27 1.27)) hide)
+    )
+    (property "JLC" "1206" (id 5) (at 83.185 320.04 0)
+      (effects (font (size 1.27 1.27)) hide)
+    )
+    (pin "1")
+    (pin "2")
+  )
   (symbol (lib_id "power:GND") (at 265.43 88.9 90) (unit 1)
     (in_bom yes) (on_board yes)
@@
       (reference "C14") (unit 1) (value "1n") (footprint "Capacitor_SMD:C_0603_1608Metric")
     )
+    (path "/e836151b-9ab0-48aa-837c-2f272734c915"
+      (reference "C15") (unit 1) (value "1n") (footprint "Capacitor_SMD:C_0603_1608Metric")
+    )
     (path "/36ea96d6-f7e9-4609-978c-86286f222fe7"

Commit message: .
Parts:
- added H1, H2: MountingHole, MountingHole:MountingHole_3.2mm_M3, symbol Mechanical:MountingHole
- added H3: MountingHole, symbol Mechanical:MountingHole
Changed lines of the file:
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@@
     (pin "1")
+  )
+  (symbol (lib_id "Mechanical:MountingHole") (at 217.17 145.415 0) (unit 1)
+    (in_bom yes) (on_board yes) (fields_autoplaced)
+    (property "Reference" "H2" (id 0) (at 219.71 144.5803 0)
+      (effects (font (size 1.27 1.27)) (justify left))
+    )
+    (property "Value" "MountingHole" (id 1) (at 219.71 147.1172 0)
+      (effects (font (size 1.27 1.27)) (justify left))
+    )
+    (property "Footprint" "MountingHole:MountingHole_3.2mm_M3" (id 2) (at 217.17 145.415 0)
+      (effects (font (size 1.27 1.27)) hide)
+    )
+    (property "Datasheet" "~" (id 3) (at 217.17 145.415 0)
+      (effects (font (size 1.27 1.27)) hide)
+    )
   )
   (symbol (lib_id "power:+5V") (at 265.43 91.44 270) (unit 1)
@@
     (pin "1")
     (pin "2")
+  )
+  (symbol (lib_id "Mechanical:MountingHole") (at 217.17 140.335 0) (unit 1)
+    (in_bom yes) (on_board yes) (fields_autoplaced)
+    (property "Reference" "H1" (id 0) (at 219.71 139.5003 0)
+      (effects (font (size 1.27 1.27)) (justify left))
+    )
+    (property "Value" "MountingHole" (id 1) (at 219.71 142.0372 0)
+      (effects (font (size 1.27 1.27)) (justify left))
+    )
+    (property "Footprint" "MountingHole:MountingHole_3.2mm_M3" (id 2) (at 217.17 140.335 0)
+      (effects (font (size 1.27 1.27)) hide)
+    )
+    (property "Datasheet" "~" (id 3) (at 217.17 140.335 0)
+      (effects (font (size 1.27 1.27)) hide)
+    )
   )
   (symbol (lib_id "Device:R") (at 160.02 172.72 180) (unit 1)
@@
     (pin "2")
   )
+  (symbol (lib_id "Mechanical:MountingHole") (at 217.17 150.495 0) (unit 1)
+    (in_bom yes) (on_board yes) (fields_autoplaced)
+    (property "Reference" "H3" (id 0) (at 219.71 149.6603 0)
+      (effects (font (size 1.27 1.27)) (justify left))
+    )
+    (property "Value" "MountingHole" (id 1) (at 219.71 152.1972 0)
+      (effects (font (size 1.27 1.27)) (justify left))
+    )
+    (property "Footprint" "" (id 2) (at 217.17 150.495 0)
+      (effects (font (size 1.27 1.27)) hide)
+    )
+    (property "Datasheet" "~" (id 3) (at 217.17 150.495 0)
+      (effects (font (size 1.27 1.27)) hide)
+    )
+  )
   (symbol (lib_id "power:GND") (at 119.38 154.94 0) (unit 1)
     (in_bom yes) (on_board yes)
@@
       (reference "F2") (unit 1) (value "550mA MT") (footprint "Fuse:Fuse_Littelfuse_372_D8.50mm")
     )
+    (path "/25215f94-21cb-4a8e-a9d7-766fb75c49cf"
+      (reference "H1") (unit 1) (value "MountingHole") (footprint "MountingHole:MountingHole_3.2mm_M3")
+    )
+    (path "/1e3a68eb-9e48-4862-aa24-b30596eab595"
+      (reference "H2") (unit 1) (value "MountingHole") (footprint "MountingHole:MountingHole_3.2mm_M3")
+    )
+    (path "/e6f01b5b-20cd-4b63-bd20-86f9fd011aaa"
+      (reference "H3") (unit 1) (value "MountingHole") (footprint "MountingHole:MountingHole_3.2mm_M3")
+    )
     (path "/ab6cb2cb-137b-41ef-bb3c-f9e222cb7a6d"

Commit message: .
Parts:
- removed C5, C6, C7, C8: 10p, Capacitor_SMD:C_0603_1608Metric, symbol Device:C_Small
- added D? (x4): ESD3.3V88D-LA, Diode_SMD:D_SOD-923, symbol Diode:ESD9B3.3ST5G
- added R?: 10k, Resistor_SMD:R_0603_1608Metric, symbol Device:R
- C3: value 22µ -> 22u
- H3: footprint (none) -> MountingHole:MountingHole_3.2mm_M3
- L1: value L -> FB0805/600R/2A
Connections:
- net 3V3-2: now also R12.2; no longer J2.11 (RLED+)
- net GND: now also D?.2 (A2), D?.2 (A2), D?.2 (A2), D?.2 (A2), R?.1; no longer R12.2
- net RX_N: now also D?.1 (A1)
- net RX_P: now also D?.1 (A1)
- net TX_N: now also D?.1 (A1)
- net TX_P: now also D?.1 (A1)
- net at R12.1: now also J2.11 (RLED+); no longer J2.12 (RLED-)
- net at U2.2 (LED2/nINTSEL): now also J2.12 (RLED-), R?.2
Other:
- moved on the sheet: C3, C4, L1, R10, R11, R12, R13, R9

Commit message: .
Parts:
- gave numbers to parts that had none: 5
