File: UniSeb32.kicad_pcb (KiCad board)
At the start: 4 copper layers, 72 x 100 mm, 57 parts, among them J1 IO, J101 Micro_SD_Card_Det, J2 ARJM11C7-114-BA-EW2, J3 Conn_02x05_Odd_Even, J6 SDS011, J7 Conn_01x02_Female, J8 Conn_01x02_Female, U1 mini_esp32, U2 LAN8720A, U3 AMS1117-3.3, U4 AMS5915, U5 module_bme280, U6 RT9400, U7 MCP23008-xSS, U8 HLK-PM01, X1 233-508, X2 233-503, X3 233-504

Commit message: .
Parts:
- added H1: MountingHole, MountingHole:MountingHole_3.2mm_M3, F.Cu at (116.8, 93.5)
- added H2: MountingHole, MountingHole:MountingHole_3.2mm_M3, F.Cu at (116.8, 131.5)
- added H3: MountingHole, MountingHole:MountingHole_3.2mm_M3, F.Cu at (180.3, 131.5)
- moved U5 0.50 mm to (177.7, 115.0)
Changed lines of the file:
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@@
   (net 81 "unconnected-(J101-Pad9)")
   (net 82 "unconnected-(J101-Pad10)")
-  (net 83 "Net-(J2-PadSH2)")
-  (net 84 "Net-(J2-PadSH1)")
+  (net 83 "Net-(C14-Pad1)")
+  (net 84 "Net-(C15-Pad1)")
   (net 85 "/TX_P")
   (net 86 "/TX_N")
@@
       (net 50 "Net-(J2-Pad14)") (pinfunction "LLED-") (pintype "passive"))
     (pad "SH1" thru_hole circle (at -7.24 5.84 180) (size 2.2 2.2) (drill 1.8) (layers *.Cu *.Mask)
-      (net 84 "Net-(J2-PadSH1)") (pinfunction "SHIELD") (pintype "passive"))
+      (net 84 "Net-(C15-Pad1)") (pinfunction "SHIELD") (pintype "passive"))
     (pad "SH2" thru_hole circle (at 8.51 5.84 180) (size 2.2 2.2) (drill 1.8) (layers *.Cu *.Mask)
-      (net 83 "Net-(J2-PadSH2)") (pinfunction "SHIELD") (pintype "passive"))
+      (net 83 "Net-(C14-Pad1)") (pinfunction "SHIELD") (pintype "passive"))
   )
   (footprint "ESP32_mini:ESP32_mini" (layer "F.Cu")
@@
   )
   (footprint "usini_sensors:module_bme280" (layer "F.Cu")
-    (at 177.67 115.464 180)
+    (at 177.67 114.964 180)
     (property "Sheetfile" "UniSeb32.kicad_sch")
     (property "Sheetname" "")
@@
     )
   )
+  (footprint "MountingHole:MountingHole_3.2mm_M3" (layer "F.Cu")
+    (at 116.7511 131.5036)
+    (descr "Mounting Hole 3.2mm, no annular, M3")
+    (tags "mounting hole 3.2mm no annular m3")
+    (property "Sheetfile" "UniSeb32.kicad_sch")
+    (property "Sheetname" "")
+    (attr exclude_from_pos_files)
+    (fp_text reference "H2" (at 0 -4.2) (layer "F.SilkS") hide
+      (effects (font (size 1 1) (thickness 0.15)))
+    )
+    (fp_text value "MountingHole" (at 0 4.2) (layer "F.Fab") hide
+      (effects (font (size 1 1) (thickness 0.15)))
+    )
+    (fp_text user "${REFERENCE}" (at 0 0) (layer "F.Fab")
+      (effects (font (size 1 1) (thickness 0.15)))
+    )
+    (fp_circle (center 0 0) (end 3.2 0) (layer "Cmts.User") (width 0.15) (fill none))
+    (fp_circle (center 0 0) (end 3.45 0) (layer "F.CrtYd") (width 0.05) (fill none))
+    (pad "" np_thru_hole circle (at 0 0) (size 3.2 3.2) (drill 3.2) (layers *.Cu *.Mask))
+  )
   (footprint "Resistor_THT:R_Axial_DIN0414_L11.9mm_D4.5mm_P5.08mm_Vertical" (layer "F.Cu")
     (at 133.858 122.411 90)
@@
     )
   )
+  (footprint "MountingHole:MountingHole_3.2mm_M3" (layer "F.Cu")
+    (at 116.7511 93.5036)
+    (descr "Mounting Hole 3.2mm, no annular, M3")
+    (tags "mounting hole 3.2mm no annular m3")
+    (property "Sheetfile" "UniSeb32.kicad_sch")
+    (property "Sheetname" "")
+    (attr exclude_from_pos_files)
+    (fp_text reference "H1" (at 0 -4.2) (layer "F.SilkS") hide
+      (effects (font (size 1 1) (thickness 0.15)))
+    )
+    (fp_text value "MountingHole" (at 0 4.2) (layer "F.Fab") hide
+      (effects (font (size 1 1) (thickness 0.15)))
+    )
+    (fp_text user "${REFERENCE}" (at 0 0) (layer "F.Fab")
+      (effects (font (size 1 1) (thickness 0.15)))
+    )
+    (fp_circle (center 0 0) (end 3.2 0) (layer "Cmts.User") (width 0.15) (fill none))
+    (fp_circle (center 0 0) (end 3.45 0) (layer "F.CrtYd") (width 0.05) (fill none))
+    (pad "" np_thru_hole circle (at 0 0) (size 3.2 3.2) (drill 3.2) (layers *.Cu *.Mask))
+  )
   (footprint "con-wago:con-wago-233-503" (layer "F.Cu")
     (at 156.2361 139.1286)
@@
     )
   )
+  (footprint "MountingHole:MountingHole_3.2mm_M3" (layer "F.Cu")
+    (at 180.2511 131.5036)
+    (descr "Mounting Hole 3.2mm, no annular, M3")
+    (tags "mounting hole 3.2mm no annular m3")
+    (property "Sheetfile" "UniSeb32.kicad_sch")
+    (property "Sheetname" "")
+    (attr exclude_from_pos_files)
+    (fp_text reference "H3" (at 0 -4.2) (layer "F.SilkS") hide
+      (effects (font (size 1 1) (thickness 0.15)))
+    )
+    (fp_text value "MountingHole" (at 0 4.2) (layer "F.Fab") hide
+      (effects (font (size 1 1) (thickness 0.15)))
+    )
+    (fp_text user "${REFERENCE}" (at 0 0) (layer "F.Fab")
+      (effects (font (size 1 1) (thickness 0.15)))
+    )
+    (fp_circle (center 0 0) (end 3.2 0) (layer "Cmts.User") (width 0.15) (fill none))
+    (fp_circle (center 0 0) (end 3.45 0) (layer "F.CrtYd") (width 0.05) (fill none))
+    (pad "" np_thru_hole circle (at 0 0) (size 3.2 3.2) (drill 3.2) (layers *.Cu *.Mask))
+  )
   (footprint "Jumper:SolderJumper-3_P1.3mm_Open_Pad1.0x1.5mm_NumberLabels" (layer "F.Cu")
     (at 117.5011 105.4736 -90)
@@
     (fp_line (start 0.8 0.4) (end 0.8 -0.4) (layer "B.Fab") (width 0.1))
     (pad "1" smd roundrect (at -0.775 0 90) (size 0.9 0.95) (layers "B.Cu" "B.Paste" "B.Mask") (roundrect_rratio 0.25)
-      (net 83 "Net-(J2-PadSH2)") (pintype "passive"))
+      (net 83 "Net-(C14-Pad1)") (pintype "passive"))
     (pad "2" smd roundrect (at 0.775 0 90) (size 0.9 0.95) (layers "B.Cu" "B.Paste" "B.Mask") (roundrect_rratio 0.25)
       (net 1 "GND") (pintype "passive"))
@@
     (fp_line (start -0.8 0.4) (end 0.8 0.4) (layer "B.Fab") (width 0.1))
     (pad "1" smd roundrect (at -0.775 0 90) (size 0.9 0.95) (layers "B.Cu" "B.Paste" "B.Mask") (roundrect_rratio 0.25)
-      (net 84 "Net-(J2-PadSH1)") (pintype "passive"))
+      (net 84 "Net-(C15-Pad1)") (pintype "passive"))
     (pad "2" smd roundrect (at 0.775 0 90) (size 0.9 0.95) (layers "B.Cu" "B.Paste" "B.Mask") (roundrect_rratio 0.25)
       (net 1 "GND") (pintype "passive"))
@@
     (effects (font (size 0.560832 0.560832) (thickness 0.048768)))
   )
-  (gr_text "extern\n5V supply" (at 117.5011 121.6661 270) (layer "F.SilkS")
+  (gr_text "extern\n5V supply" (at 117.5 121.25 270) (layer "F.SilkS")
     (effects (font (size 0.93472 0.93472) (thickness 0.08128)) (justify left))
   )
@@
   (segment (start 122.6611 107.3786) (end 122.6611 114.1211) (width 0.8128) (layer "F.Cu") (net 9))
   (segment (start 117.5011 105.4736) (end 120.7561 105.4736) (width 0.8128) (layer "F.Cu") (net 9))
-  (segment (start 181.08 136.122) (end 181.08 139) (width 0.254) (layer "F.Cu") (net 10))
-  (segment (start 174.752 124.714) (end 176.657 126.619) (width 0.254) (layer "F.Cu") (net 10))
-  (segment (start 176.657 126.619) (end 176.657 131.699) (width 0.254) (layer "F.Cu") (net 10))
-  (segment (start 176.657 131.699) (end 181.08 136.122) (width 0.254) (layer "F.Cu") (net 10))
+  (segment (start 181.08 138.101) (end 181.08 139) (width 0.254) (layer "F.Cu") (net 10))
+  (segment (start 174.752 124.714) (end 176 125.962) (width 0.254) (layer "F.Cu") (net 10))
+  (segment (start 176 125.962) (end 176 133.021) (width 0.254) (layer "F.Cu") (net 10))
+  (segment (start 176 133.021) (end 181.08 138.101) (width 0.254) (layer "F.Cu") (net 10))
   (via (at 174.752 124.714) (size 0.8) (drill 0.4) (layers "F.Cu" "B.Cu") (net 10))
   (segment (start 174.752 120.269) (end 167.717 113.234) (width 0.254) (layer "B.Cu") (net 10))
   (segment (start 174.752 124.714) (end 174.752 120.269) (width 0.254) (layer "B.Cu") (net 10))
   (segment (start 167.717 113.234) (end 167.717 111.464) (width 0.254) (layer "B.Cu") (net 10))
+  (segment (start 175.26 133.51) (end 178.54 136.79) (width 0.254) (layer "F.Cu") (net 11))
+  (segment (start 178.54 136.79) (end 178.54 139) (width 0.254) (layer "F.Cu") (net 11))
+  (segment (start 175.26 127.254) (end 175.26 133.51) (width 0.254) (layer "F.Cu") (net 11))
   (segment (start 173.736 125.73) (end 175.26 127.254) (width 0.254) (layer "F.Cu") (net 11))
-  (segment (start 178.54 135.36) (end 178.54 139) (width 0.254) (layer "F.Cu") (net 11))
-  (segment (start 175.26 127.254) (end 175.26 132.08) (width 0.254) (layer "F.Cu") (net 11))
-  (segment (start 175.26 132.08) (end 178.54 135.36) (width 0.254) (layer "F.Cu") (net 11))
   (via (at 173.736 125.73) (size 0.8) (drill 0.4) (layers "F.Cu" "B.Cu") (net 11))
   (segment (start 173.736 125.73) (end 173.736 120.269) (width 0.254) (layer "B.Cu") (net 11))
